Commit message: feat: 提交可用的右臂urdf

File: robot_description/biped_s49_description/urdf/biped_s49_right_arm.urdf (robot description, URDF)
Before this commit: robot biped_s49_right_arm, 10 links, 9 joints
Links:
- added link camera, mass 0.0497265773443356; visual mesh filename=package://kuavo_assets/models/biped_s49/meshes/camera.STL
- added link camera_base, mass 0.0000392699081698732; visual mesh filename=package://kuavo_assets/models/biped_s49/meshes/camera_base.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
- added link l_hand_camera, mass 0.038145442577304; visual mesh filename=package://kuavo_assets/models/biped_s49/meshes/l_hand_camer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
- added link l_hand_tripod, mass 0.0342669089979502; visual mesh filename=package://kuavo_assets/models/biped_s49/meshes/l_hand_tripo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
- added link leg_l1_link, mass 1.71093115; visual mesh filename=package://kuavo_assets/models/biped_s49/meshes/l_leg_roll.S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
- added link leg_l2_link, mass 0.58029165; visual mesh filename=package://kuavo_assets/models/biped_s49/meshes/l_leg_yaw.STL
- added link leg_l3_link, mass 4.50393141; visual mesh filename=package://kuavo_assets/models/biped_s49/meshes/l_leg_pitch.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
- added link leg_l4_link, mass 1.62776815; visual mesh filename=package://kuavo_assets/models/biped_s49/meshes/l_knee.STL
- added link leg_l5_link, mass 0.07193524; visual mesh filename=package://kuavo_assets/models/biped_s49/meshes/l_foot_pitch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
- added link leg_l6_link, mass 0.49861272; collision box size=0.25 0.1 0.04; visual mesh filename=package://kuavo_assets/models/biped_s49/meshes/l_foot_roll.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
- added link leg_r1_link, mass 1.71093008; visual mesh filename=package://kuavo_assets/models/biped_s49/meshes/r_leg_roll.S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
- added link leg_r2_link, mass 0.58029165; visual mesh filename=package://kuavo_assets/models/biped_s49/meshes/r_leg_yaw.STL
- added link leg_r3_link, mass 4.50385993; visual mesh filename=package://kuavo_assets/models/biped_s49/meshes/r_leg_pitch.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
- added link leg_r4_link, mass 1.62655699; visual mesh filename=package://kuavo_assets/models/biped_s49/meshes/r_knee.STL
- added link leg_r5_link, mass 0.07193524; visual mesh filename=package://kuavo_assets/models/biped_s49/meshes/r_foot_pitch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
- added link leg_r6_link, mass 0.49861272; visual mesh filename=package://kuavo_assets/models/biped_s49/meshes/r_foot_roll.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
- added link r_hand_camera, mass 0.038145442577304; visual mesh filename=package://kuavo_assets/models/biped_s49/meshes/r_hand_camer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
- added link r_hand_tripod, mass 0.034266881719861; visual mesh filename=package://kuavo_assets/models/biped_s49/meshes/r_hand_tripo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
- added link radar, mass 0.149896342265089; visual mesh filename=package://kuavo_assets/models/biped_s49/meshes/radar.STL
- added link zarm_l1_link, mass 0.95200000; collision cylinder length=0.04 radius=0.05; visual mesh filename=package://kuavo_assets/models/biped_s49/meshes/l_arm_pitch.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
- added link zarm_l2_link, mass 0.38500000; visual mesh filename=package://kuavo_assets/models/biped_s49/meshes/l_arm_roll.S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
- added link zarm_l3_link, mass 1.75450000; collision cylinder length=0.14 radius=0.045; visual mesh filename=package://kuavo_assets/models/biped_s49/meshes/l_arm_yaw.STL
- added link zarm_l4_link, mass 0.60780000; collision cylinder length=0.18 radius=0.045; visual mesh filename=package://kuavo_assets/models/biped_s49/meshes/l_forearm.STL
- added link zarm_l5_link, mass 0.63690000; visual mesh filename=package://kuavo_assets/models/biped_s49/meshes/l_hand_yaw.S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
- added link zarm_l6_link, mass 0.47390000; visual mesh filename=package://kuavo_assets/models/biped_s49/meshes/l_hand_roll.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
- added link zarm_l7_end_effector
- added link zarm_l7_link, mass 0.7374; collision box size=0.08 0.05 0.16; collision cylinder length=0.08 radius=0.01
- added link zhead_1_link, mass 0.35; visual mesh filename=package://kuavo_assets/models/biped_s49/meshes/head_yaw.STL
- added link zhead_2_link, mass 0.5492; visual mesh filename=package://kuavo_assets/models/biped_s49/meshes/head_pitch.S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
- link zarm_r1_link: geometry visual mesh filename=package://kuavo_assets/models/biped_s49/meshes/r_arm_pitch.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
- link zarm_r3_link: geometry visual mesh filename=package://kuavo_assets/models/biped_s49/meshes/r_arm_yaw.STL
- link zarm_r4_link: geometry visual mesh filename=package://kuavo_assets/models/biped_s49/meshes/r_forearm.STL
- link zarm_r7_link: mass 0.0542110173081966 -> 0.7374; geometry visual mesh filename=package://kuavo_assets/models/biped_s49/meshes/r_hand_pitch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
Joints:
- added joint camera: type fixed, parent zhead_2_link, child camera, origin xyz=0.102420738776518 -0.0475000000000003 0.126192926717169 rpy=3.14159265358979 0.383972435438723 0
- added joint camera_base: type fixed, parent zhead_2_link, child camera_base, origin xyz=0.0932759773834307 0 0.145322661773667 rpy=3.14159265358979 0.383972435438723 0
- added joint l_hand_camera_joint: type fixed, parent l_hand_tripod, child l_hand_camera, origin xyz=0.11540559159102 -0.0145586110669961 -0.110123491595499 rpy=1.919862177193763 0.753528063917894 -2.897246568680842, axis 0 0 0
- added joint l_hand_tripod_joint: type fixed, parent zarm_l7_link, child l_hand_tripod, origin xyz=0.0 0.0 0.0 rpy=0.0 0.0 0.0, axis 0 0 0
- added joint leg_l1_joint: type fixed, parent base_link, child leg_l1_link, origin xyz=-0.0024999 0.087 -0.066 rpy=0 0 0, axis 1 0 0, limit lower=-0.314159265358979 upper=0.663225115757845 effort=180.0 velocity=10.46
- added joint leg_l2_joint: type fixed, parent leg_l1_link, child leg_l2_link, origin xyz=0 0 0 rpy=0 0 0, axis 0 0 1, limit lower=-0.872664625997165 upper=0.785398163397448 effort=22.2 velocity=10.46
- added joint leg_l3_joint: type fixed, parent leg_l2_link, child leg_l3_link, origin xyz=0.000500354536093913 -0.00100000000000011 -0.1287 rpy=0 0 0, axis 0 1 0, limit lower=-2.00712863979348 upper=1.5707963267949 effort=72.0 velocity=20.93
- added joint leg_l4_joint: type fixed, parent leg_l3_link, child leg_l4_link, origin xyz=-6.87185435835039E-05 0 -0.284 rpy=0 0 0, axis 0 1 0, limit lower=0.0 upper=2.53072741539178 effort=135.0 velocity=11.62
- added joint leg_l5_joint: type fixed, parent leg_l4_link, child leg_l5_link, origin xyz=-0.000431635992531742 0 -0.346000000000001 rpy=0 0 0, axis 0 1 0, limit lower=-0.872664625997165 upper=0.349065850398866 effort=46.0 velocity=10.46
- added joint leg_l6_joint: type fixed, parent leg_l5_link, child leg_l6_link, origin xyz=0 0 0 rpy=0 0 0, axis 1 0 0, limit lower=-0.261799387799149 upper=0.261799387799149 effort=30.0 velocity=10.46
- added joint leg_r1_joint: type fixed, parent base_link, child leg_r1_link, origin xyz=-0.0024999 -0.087 -0.066 rpy=0 0 0, axis 1 0 0, limit lower=-0.663225115757845 upper=0.314159265358979 effort=127.0 velocity=10.46
- added joint leg_r2_joint: type fixed, parent leg_r1_link, child leg_r2_link, origin xyz=0 0 0 rpy=0 0 0, axis 0 0 1, limit lower=-0.785398163397448 upper=0.872664625997165 effort=22.2 velocity=10.46
- added joint leg_r3_joint: type fixed, parent leg_r2_link, child leg_r3_link, origin xyz=-4.88006581312577E-05 0 -0.1287 rpy=0 0 0, axis 0 1 0, limit lower=-2.00712863979348 upper=1.5707963267949 effort=72.0 velocity=20.93
- added joint leg_r4_joint: type fixed, parent leg_r3_link, child leg_r4_link, origin xyz=0.000147138572785148 0 -0.283999982974744 rpy=0 0 0, axis 0 1 0, limit lower=0.0 upper=2.53072741539178 effort=135.0 velocity=11.62
- added joint leg_r5_joint: type fixed, parent leg_r4_link, child leg_r5_link, origin xyz=0.000119806050928577 0 -0.345999979257963 rpy=0 0 0, axis 0 1 0, limit lower=-0.872664625997165 upper=0.349065850398866 effort=46.0 velocity=10.46
- added joint leg_r6_joint: type fixed, parent leg_r5_link, child leg_r6_link, origin xyz=0 0 0 rpy=0 0 0, axis 1 0 0, limit lower=-0.261799387799149 upper=0.261799387799149 effort=30.0 velocity=10.46
- added joint r_hand_camera_joint: type fixed, parent r_hand_tripod, child r_hand_camera, origin xyz=0.115405591590931 0.0154312352120435 -0.107724128430896 rpy=1.208853693239594  0.751879414295006 2.888346587751982, axis 0 0 0
- added joint r_hand_tripod_joint: type fixed, parent zarm_r7_link, child r_hand_tripod, origin xyz=0.0 0.0 0.0 rpy=0.0 0.0 0.0, axis 0 0 0
- added joint radar: type fixed, parent zhead_2_link, child radar, origin xyz=0.0217799337881943 0 0.105417258037133 rpy=0 0.229686043245049 0
- added joint zarm_l1_joint: type fixed, parent base_link, child zarm_l1_link, origin xyz=-0.017499853 0.29269999999999996 0.4245 rpy=0 0 0, axis 0 1 0, limit lower=-2.94159265358979 upper=0.0 effort=66.67 velocity=2.0
- added joint zarm_l2_joint: type fixed, parent zarm_l1_link, child zarm_l2_link, origin xyz=0 0 0 rpy=0 0 0, axis 1 0 0, limit lower=0.0 upper=1.8943951023932 effort=75.0 velocity=2.0
- added joint zarm_l3_joint: type fixed, parent zarm_l2_link, child zarm_l3_link, origin xyz=0 0 0 rpy=0 0 0, axis 0 0 1, limit lower=-0.387 upper=1.3707963267949 effort=57.0 velocity=2.0
- added joint zarm_l4_joint: type fixed, parent zarm_l3_link, child zarm_l4_link, origin xyz=0.0200000000000006 0 -0.283699999999996 rpy=0 0 0, axis 0 1 0, limit lower=-2.1 upper=-0.2 effort=75.0 velocity=2.0
- added joint zarm_l5_joint: type fixed, parent zarm_l4_link, child zarm_l5_link, origin xyz=-0.0200000000000025 0 -0.127037274261591 rpy=0 0 0, axis 0 0 1, limit lower=-1.3707963267949 upper=1.3707963267949 effort=14.1 velocity=5.5
- added joint zarm_l6_joint: type fixed, parent zarm_l5_link, child zarm_l6_link, origin xyz=0.000199999999999079 0 -0.106462725738415 rpy=0 0 0, axis 1 0 0, limit lower=-1.013 upper=0.598131700797732 effort=14.1 velocity=5.5
- added joint zarm_l7_end_effector_joint: type fixed, parent zarm_l7_link, child zarm_l7_end_effector, origin xyz=0 -0.03 -0.17 rpy=0 0 0
- added joint zarm_l7_joint: type fixed, parent zarm_l6_link, child zarm_l7_link, origin xyz=0 0 -0.0210004653879916 rpy=0 0 0, axis 0 1 0, limit lower=-0.498131700797732 upper=0.498131700797732 effort=14.1 velocity=5.5
- added joint zhead_1_joint: type fixed, parent base_link, child zhead_1_link, origin xyz=-0.018499853 0.0 0.6014 rpy=0 0 0, axis 0 0 1, limit lower=-1.5707963267949 upper=1.5707963267949 effort=1.5 velocity=5.23333333333333
- added joint zhead_2_joint: type fixed, parent zhead_1_link, child zhead_2_link, origin xyz=0 0 0 rpy=0 0 0, axis 0 1 0, limit lower=-0.523598775598299 upper=0.523598775598299 effort=12.0 velocity=5.23333333333333
- joint zarm_r1_joint: limit lower=0.0 upper=2.8159265358979 effort=66.67 velocity=2.0 -> lower=-2.94159265358979 upper=0.0 effort=66.67 velocity=2.0
- joint zarm_r3_joint: limit lower=-1.4907963267949 upper=0.287 effort=57.0 velocity=3.0 -> lower=1.3707963267949 upper=-0.387 effort=57.0 velocity=2.0
- joint zarm_r4_joint: limit lower=-0.1 upper=2.0 effort=75.0 velocity=3.0 -> lower=-2.1 upper=-0.2 effort=75.0 velocity=2.0; origin xyz=0.0200000000000006 0 -0.283699999999996 rpy=0 0 0 -> xyz=0.0200000000000024 0 -0.2837 rpy=0 0 0
- joint zarm_r5_joint: limit lower=-1.4007963267949 upper=1.4007963267949 effort=14.1 velocity=5.5 -> lower=-1.3707963267949 upper=1.3707963267949 effort=14.1 velocity=5.5; origin xyz=-0.0200000000000025 0 -0.127037274261591 rpy=0 0 0 -> xyz=-0.0200000000000001 0 -0.127037274261587 rpy=0 0 0
- joint zarm_r6_joint: limit lower=-0.598131700797732 upper=0.713 effort=14.1 velocity=5.5 -> lower=-0.598131700797732 upper=1.013 effort=14.1 velocity=5.5; origin xyz=0.000199999999999079 0 -0.106462725738415 rpy=0 0 0 -> xyz=0 0 -0.106462725738415 rpy=0 0 0
- joint zarm_r7_joint: limit lower=-0.598131700797732 upper=0.598131700797732 effort=14.1 velocity=5.5 -> lower=-0.498131700797732 upper=0.498131700797732 effort=14.1 velocity=5.5; origin xyz=0 0 -0.0210004653879916 rpy=0 0 0 -> xyz=0 0 -0.0209999999999999 rpy=0 0 0
