Commit message: fix: 调整ar5的关节速度限制

File: robot_description/ar5_tutorial/urdf/ar5_leftArm.urdf (robot description, URDF)
Before this commit: robot robot, 20 links, 19 joints
Joints:
- joint AR5-5_07L-W4C4A2_joint_1: limit lower=-3.1067 upper=0.0 effort=108 velocity=3.0543261909900763 -> lower=-3.1067 upper=0.0 effort=108 velocity=2.0543261909900763
- joint AR5-5_07L-W4C4A2_joint_2: limit lower=-2.0944 upper=0.0 effort=108 velocity=3.0543261909900763 -> lower=-2.0944 upper=0.0 effort=108 velocity=2.0543261909900763
- joint AR5-5_07L-W4C4A2_joint_3: limit lower=-3.1067 upper=-1.1838 effort=66 velocity=4.71238898038469 -> lower=-3.1067 upper=-1.1838 effort=66 velocity=2.01238898038469
- joint AR5-5_07L-W4C4A2_joint_4: limit lower=0.0 upper=2.1 effort=66 velocity=5.235987755982989 -> lower=0.0 upper=2.1 effort=66 velocity=2.035987755982989
- joint AR5-5_07R-W4C4A2_joint_1: limit lower=-3.1067 upper=3.1067 effort=108 velocity=3.0543261909900763 -> lower=-3.1067 upper=3.1067 effort=108 velocity=2.0543261909900763
- joint AR5-5_07R-W4C4A2_joint_2: limit lower=-2.0944 upper=2.0944 effort=108 velocity=3.0543261909900763 -> lower=-2.0944 upper=2.0944 effort=108 velocity=2.0543261909900763
- joint AR5-5_07R-W4C4A2_joint_3: limit lower=-3.1067 upper=3.1067 effort=66 velocity=4.71238898038469 -> lower=-3.1067 upper=3.1067 effort=66 velocity=2.01238898038469
- joint AR5-5_07R-W4C4A2_joint_4: limit lower=-1.0472 upper=2.5307 effort=66 velocity=5.235987755982989 -> lower=-1.0472 upper=2.5307 effort=66 velocity=2.035987755982989

File: robot_description/ar5_tutorial/urdf/ar5_rightArm.urdf (robot description, URDF)
Before this commit: robot robot, 20 links, 19 joints
Joints:
- joint AR5-5_07L-W4C4A2_joint_1: limit lower=-3.1067 upper=3.1067 effort=108 velocity=3.0543261909900763 -> lower=-3.1067 upper=3.1067 effort=108 velocity=2.0543261909900763
- joint AR5-5_07L-W4C4A2_joint_2: limit lower=-2.0944 upper=2.0944 effort=108 velocity=3.0543261909900763 -> lower=-2.0944 upper=2.0944 effort=108 velocity=2.0543261909900763
- joint AR5-5_07L-W4C4A2_joint_3: limit lower=-3.1067 upper=3.1067 effort=66 velocity=4.71238898038469 -> lower=-3.1067 upper=3.1067 effort=66 velocity=2.01238898038469
- joint AR5-5_07L-W4C4A2_joint_4: limit lower=-1.0472 upper=2.5307 effort=66 velocity=5.235987755982989 -> lower=-1.0472 upper=2.5307 effort=66 velocity=2.01238898038469
- joint AR5-5_07R-W4C4A2_joint_1: limit lower=0.0 upper=3.1067 effort=108 velocity=3.0543261909900763 -> lower=0.0 upper=3.1067 effort=108 velocity=2.0543261909900763
- joint AR5-5_07R-W4C4A2_joint_2: limit lower=-2.0944 upper=0.0 effort=108 velocity=3.0543261909900763 -> lower=-2.0944 upper=0.0 effort=108 velocity=2.0543261909900763
- joint AR5-5_07R-W4C4A2_joint_3: limit lower=1.1838 upper=3.1067 effort=66 velocity=4.71238898038469 -> lower=1.1838 upper=3.1067 effort=66 velocity=2.01238898038469
- joint AR5-5_07R-W4C4A2_joint_4: limit lower=0.0 upper=2.1 effort=66 velocity=5.235987755982989 -> lower=0.0 upper=2.1 effort=66 velocity=2.035987755982989

Commit message: fix: 调整 ar5 模型，对齐最新构型和零点

File: robot_description/ar5_tutorial/urdf/ar5_leftArm.urdf (robot description, URDF)
Before this commit: robot robot, 20 links, 19 joints
Links:
- removed link world
- added link base_link
- link torso: geometry visual mesh filename=package://ar5_tutorial/meshes/base.stl scale=0.0008 0.0008 0.0008
Joints:
- joint AR5-5_07L-W4C4A2_joint_1: limit lower=-3.1067 upper=0.0 effort=108 velocity=2.0543261909900763 -> lower=-3.1067 upper=0.0 effort=108 velocity=3.0543261909900763
- joint AR5-5_07L-W4C4A2_joint_2: axis 0 1 0 -> 0 -1 0; limit lower=-2.0944 upper=0.0 effort=108 velocity=2.0543261909900763 -> lower=0.0 upper=2.0944 effort=108 velocity=3.0543261909900763
- joint AR5-5_07L-W4C4A2_joint_3: limit lower=-3.1067 upper=-1.1838 effort=66 velocity=2.01238898038469 -> lower=-1.5359 upper=0.7 effort=66 velocity=4.71238898038469; origin xyz=0.0 0.0 0.314 rpy=0 0 0 -> xyz=0.0 0.0 0.314 rpy=0 0 -1.570796
- joint AR5-5_07L-W4C4A2_joint_4: axis 0 1 0 -> 0 -1 0; limit lower=0.0 upper=2.1 effort=66 velocity=2.035987755982989 -> lower=-2.1 upper=0.0 effort=66 velocity=2.035987755982989
- joint AR5-5_07L-W4C4A2_joint_6: axis 0 1 0 -> 0 -1 0
- joint AR5-5_07R-W4C4A2_joint_2: axis 0 1 0 -> 0 -1 0
- joint AR5-5_07R-W4C4A2_joint_3: limit lower=-3.1067 upper=3.1067 effort=66 velocity=2.01238898038469 -> lower=-4.6774 upper=1.5359 effort=66 velocity=2.01238898038469; origin xyz=0.0 0.0 0.314 rpy=0 0 0 -> xyz=0.0 0.0 0.314 rpy=0 0 1.570796
- joint AR5-5_07R-W4C4A2_joint_7: axis 1 0 0 -> -1 0 0
- joint torso_base_joint: parent world -> base_link

File: robot_description/ar5_tutorial/urdf/ar5_rightArm.urdf (robot description, URDF)
Before this commit: robot robot, 20 links, 19 joints
Links:
- removed link world
- added link base_link
- link torso: geometry visual mesh filename=package://ar5_tutorial/meshes/base.stl scale=0.0008 0.0008 0.0008
Joints:
- joint AR5-5_07L-W4C4A2_joint_2: axis 0 1 0 -> 0 -1 0
- joint AR5-5_07L-W4C4A2_joint_3: limit lower=-3.1067 upper=3.1067 effort=66 velocity=2.01238898038469 -> lower=-1.5359 upper=4.6774 effort=66 velocity=2.01238898038469; origin xyz=0.0 0.0 0.314 rpy=0 0 0 -> xyz=0.0 0.0 0.314 rpy=0 0 -1.570796
- joint AR5-5_07L-W4C4A2_joint_4: axis 0 1 0 -> 0 -1 0; limit lower=-1.0472 upper=2.5307 effort=66 velocity=2.01238898038469 -> lower=-2.5307 upper=1.0472 effort=66 velocity=2.01238898038469
- joint AR5-5_07L-W4C4A2_joint_6: axis 0 1 0 -> 0 -1 0
- joint AR5-5_07R-W4C4A2_joint_2: axis 0 1 0 -> 0 -1 0; limit lower=-2.0944 upper=0.0 effort=108 velocity=2.0543261909900763 -> lower=0.0 upper=2.0944 effort=108 velocity=2.0543261909900763
- joint AR5-5_07R-W4C4A2_joint_3: limit lower=1.1838 upper=3.1067 effort=66 velocity=2.01238898038469 -> lower=-0.7 upper=1.5359 effort=66 velocity=2.01238898038469; origin xyz=0.0 0.0 0.314 rpy=0 0 0 -> xyz=0.0 0.0 0.314 rpy=0 0 1.570796
- joint AR5-5_07R-W4C4A2_joint_7: axis 1 0 0 -> -1 0 0
- joint torso_base_joint: parent world -> base_link
