Commit message: fix: 调整天机右臂的辨识关节限制

File: robot_description/marvinM6_description/marvinM6_right.urdf (robot description, URDF)
Before this commit: robot marvinM6_right, 19 links, 18 joints
Joints:
- joint Joint5_R: limit lower=-3.1067 upper=3.1067 effort=18 velocity=3.1416 -> lower=-2.1067 upper=2.1067 effort=18 velocity=3.1416
- joint Joint6_R: limit lower=-1.0472 upper=1.0472 effort=18 velocity=3.1416 -> lower=-0.7472 upper=0.7472 effort=18 velocity=3.1416
- joint Joint7_R: limit lower=-1.570796327 upper=1.570796327 effort=18 velocity=3.1416 -> lower=-0.770796327 upper=0.770796327 effort=18 velocity=3.1416
